File: pcb/Hackpad_highway.kicad_pcb (KiCad board)
At the start: 2 copper layers, 83 x 47.2 mm, 7 parts, among them SW1 SW_Push, SW2 SW_Push, SW3 SW_Push, SW4 SW_Push, U1 XIAO-RP2040-DIP

Commit message: rehaul
Connections:
- D1 pad 2: +5V -> GND
- D1 pad 4: GND -> +5V
- D2 pad 2: +5V -> GND
- D2 pad 4: GND -> +5V
Routing:
- net GND: track 288.4 -> 146.3 mm
- net Net-(U1-GPIO3/MOSI): track 27.8 -> 64.5 mm
- net Net-(U1-GPIO2/SCK): track 27.6 -> 38.9 mm
- net Net-(D1-DIN): track 21.6 -> 16.5 mm
- net +5V: track 61.1 -> 56.7 mm, vias 1 -> 2
- net Net-(D1-DOUT): track 60.2 -> 55.8 mm
- net Net-(U1-GPIO1/RX): track 46.8 -> 46.4 mm, vias 0 -> 2
Other:
- board text added: "AESTHETIC DESIGN"
- board text added: "CUSTOMIZABLE BUTTONS"
- board text added: "D-MACROPAD Like a d-pad, but a macropad."
- board text added: "FOR HIGHWAY 2025"
- board text added: "MADE BY JAYDEN L."
- board text added: "SULTANS OF SWING a.k.a. the best song ever made PLAY IT USING THE D-MACROPAD!"
- board text added: "USB-C CONNECTIVITY"
- board text added: "XIAO HERE"
- board text removed: "JAYDEN'S D-MACROPAD"
- board text removed: "XIAO HERE!"
